File: PowerManagment/PowerMangment/_autosave-PowerMangment.kicad_sch (KiCad schematic)
At the start: 14 parts, among them J1 Barrel_Jack_Switch, J2 USB_B_Micro, Q1 IRF4905, U1 TP4056(Module), U2 MT3608(Module), U3 MCP6024

Commit message: PowerManagment changes
Other:
- note added: "1.5V When 3.2V (Discharge) //TODO Calcs"
- note removed: "2V When 3.2V (Discharge)"
Changed lines of the file:
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@@
     (effects (font (size 3 3) (thickness 1) bold) (justify left bottom))
   )
-  (text "2V When 3.2V (Discharge)" (at 149.225 94.615 0)
+  (text "1.5V When 3.2V (Discharge) //TODO Calcs" (at 149.225 94.615 0)
     (effects (font (size 1.27 1.27)) (justify left bottom))
   )
